File: Hardware/Dom-Turretto-Hat/Dom-Turretto-Hat.kicad_pcb (KiCad board)
At the start: 2 copper layers, 65 x 56 mm, 54 parts, among them J1 Raspberry_Pi_2_3, J2 Conn_Coaxial, J3 Barrel_Jack_Switch, J4 Conn_01x02, U1 CAT24C32WI-GT3, U2 MAX-M8Q, U3 LM22679TJ-5.0/NOPB, U4 LTC4451AV#TRMPBF, U5 LTC4451AV#TRMPBF, U6 LT1963AxST-3.3, U7 LTC4411ES5TRMPBF

Commit message: Initial Layout
Parts:
- moved U4 195.6 mm to (146.2, 116.5), turned to -90 degrees
- moved J4 183.3 mm to (151.5, 121.9)
- moved U6 179.0 mm to (130.0, 114.2)
- moved C11 178.0 mm to (124.8, 113.0), turned to 90 degrees
- moved C12 177.2 mm to (124.8, 116.0), turned to -90 degrees
- moved C13 174.6 mm to (123.2, 116.0), turned to 90 degrees
- moved C9 174.0 mm to (144.2, 114.2), turned to 180 degrees
- moved J3 172.8 mm to (139.2, 119.7)
- moved C5 171.2 mm to (149.8, 116.5), turned to 180 degrees
- moved U5 170.4 mm to (142.0, 116.5), turned to 90 degrees
- moved C6 163.0 mm to (139.2, 116.5), turned to 90 degrees
- moved EXT_POW1 161.3 mm to (119.2, 97.8), turned to 180 degrees
- moved PI_POW1 161.1 mm to (118.5, 109.8), turned to -90 degrees
- moved R6 161.0 mm to (119.2, 99.3), turned to 180 degrees
- moved R7 159.5 mm to (120.0, 109.8), turned to -90 degrees
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Other:
- outline, holes or cut-outs redrawn
