File: Hardware/Dom-Turretto-Hat/Dom-Turretto-Hat.kicad_pcb (KiCad board)
At the start: 2 copper layers, 65 x 56 mm, 47 parts, among them J1 Raspberry_Pi_2_3, J2 Conn_01x02, J3 Barrel_Jack_Switch, Q1 SI4143DY-T1-GE3, Q2 SI4143DY-T1-GE3, U1 CAT24C32WI-GT3, U2 LM22679TJ-5.0/NOPB, U3 LTC4412xS6, U4 LTC4411ES5TRMPBF

Commit message: Made layout logical
Parts:
- moved R_Opt2 17.6 mm to (148.5, 130.5)
- moved R3 16.3 mm to (137.5, 113.5)
- moved R_Opt6 16.1 mm to (148.5, 126.5)
- moved R_Opt4 14.5 mm to (148.5, 122.5)
- moved C4 11.4 mm to (130.1, 98.4), turned to -90 degrees
- moved C6 11.1 mm to (122.5, 116.5), turned to 180 degrees
- moved C2 8.02 mm to (121.4, 103.8), turned to 0 degrees
- moved C1 6.06 mm to (121.4, 105.4), turned to 0 degrees
- moved C3 6.02 mm to (121.4, 102.3), turned to 0 degrees
- moved D1 4.26 mm to (126.8, 103.8)
- moved A1 4.08 mm to (166.2, 132.1)
- moved R_Opt3 3.62 mm to (149.3, 106.4)
- moved C7 3.58 mm to (140.7, 114.5)
- moved R_Opt7 2.37 mm to (149.3, 102.5)
- moved J3 2.16 mm to (138.9, 120.2)
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
Commit message: Did first draft
Parts:
- moved C7 9.04 mm to (135.0, 121.5), turned to -90 degrees
- moved R_Opt2 3.40 mm to (148.5, 127.1)
- moved R_Opt4 3.40 mm to (148.5, 119.1)
- moved R_Opt6 3.40 mm to (148.5, 123.1)
- moved C10 1.30 mm to (117.5, 88.3)
- moved EXT_POW1 1.22 mm to (136.5, 86.5)
- moved U4 1.03 mm to (121.2, 87.5)
- moved R_Opt1 0.86 mm to (142.5, 87.5), turned to 0 degrees
- moved C9 0.85 mm to (124.8, 87.5)
- moved PI_POW1 0.81 mm to (114.8, 88.5)
- moved R5 0.75 mm to (114.8, 86.5)
- moved R4 0.73 mm to (136.5, 88.5)
Routing:
- net VCC: track 0.00 -> 120.6 mm
- net /Dir1: track 0.00 -> 66.6 mm
- net /Step1: track 0.00 -> 55.8 mm
- net /Power/5V_out: track 0.00 -> 41.4 mm
- net /Step2: track 0.00 -> 41.0 mm
- net +3V3: track 0.00 -> 33.5 mm, vias 0 -> 6
- net /Dir2: track 0.00 -> 32.4 mm
- net Net-(C6-Pad1): track 0.00 -> 19.0 mm
- net Net-(Q2-Pad4): track 0.00 -> 18.1 mm, vias 0 -> 2
- net GND: track 0.00 -> 17.2 mm, vias 0 -> 1
- net +5V: track 0.00 -> 15.8 mm
- net Net-(A2-Pad12): track 0.00 -> 13.5 mm
- net /ID_SCL_EEPROM: track 0.00 -> 13.5 mm
- net Net-(Q1-Pad4): track 0.00 -> 12.9 mm
- net Net-(A2-Pad11): track 0.00 -> 12.6 mm
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- added copper zone on B.Cu, net +3V3
- added copper zone on F.Cu, net GND
- removed copper zone on B.Cu, net GND
