File: Hardware/Dom-Turretto-Hat/Dom-Turretto-Hat.kicad_pcb (KiCad board)
At the start: 2 copper layers, 65 x 56 mm, 47 parts, among them J1 Raspberry_Pi_2_3, J2 Conn_01x02, J3 Barrel_Jack_Switch, Q1 SI4143DY-T1-GE3, Q2 SI4143DY-T1-GE3, U1 CAT24C32WI-GT3, U2 LM22679TJ-5.0/NOPB, U3 LTC4412xS6, U4 LTC4411ES5TRMPBF

Commit message: Added some memes
Other:
- board text added: "Omg what are you doing stepper driver"
- board text added: "T H I C C"
Changed lines of the file:
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@@
     (property "Sheetname" "")
     (attr exclude_from_pos_files)
-    (fp_text reference "H5" (at 57.31 -6.94) (layer "F.SilkS")
+    (fp_text reference "H5" (at 0 -3.5) (layer "F.SilkS")
       (effects (font (size 1 1) (thickness 0.15)))
     )
@@
       (effects (font (size 1 1) (thickness 0.15)) (justify mirror))
     )
-    (fp_text value "Raspberry_Pi_2_3" (at -4.52 -114.03 90) (layer "B.Fab")
+    (fp_text value "Raspberry_Pi_2_3" (at -5.79 2.9 90) (layer "B.Fab")
       (effects (font (size 1 1) (thickness 0.15)) (justify mirror))
     )
@@
   (gr_arc (start 176.5 130.5) (mid 175.474874 132.974874) (end 173 134) (layer "Edge.Cuts") (width 0.1))
   (gr_line (start 156.5 134.25) (end 156.5 134) (layer "User.6") (width 0.15))
+  (gr_text "Omg what are you \ndoing stepper driver" (at 159.5 123 90) (layer "F.SilkS")
+    (effects (font (size 1 1) (thickness 0.15)))
+  )
+  (gr_text "T H I C C" (at 138.5 106) (layer "F.SilkS")
+    (effects (font (size 1 1) (thickness 0.15) italic))
+  )
   (segment (start 149.475 79.025) (end 149.145001 79.354999) (width 0.25) (layer "F.Cu") (net 1))
   (segment (start 135.225 122.5) (end 135 122.275) (width 1.1) (layer "F.Cu") (net 1))

Commit message: Made better
Parts:
- removed C11, C12: 47uF, Capacitor_SMD:CP_Elec_6.3x7.7
- added Fan1: Conn_01x02_Male, Connector_PinHeader_2.54mm:PinHeader_1x02_P2.54mm_Vertical, F.Cu at (171.8, 109.9)
- added TP1: Step1, TestPoint:TestPoint_Pad_1.5x1.5mm, F.Cu at (158.2, 128.0)
- added TP2: Step2, TestPoint:TestPoint_Pad_1.5x1.5mm, B.Cu at (146.5, 109.2)
- added TP3: Dir1, TestPoint:TestPoint_Pad_1.5x1.5mm, F.Cu at (158.2, 131.8)
- added TP4: Dir2, TestPoint:TestPoint_Pad_1.5x1.5mm, B.Cu at (149.8, 109.2)
- added TP5: SDA_EEPROM, TestPoint:TestPoint_Pad_1.5x1.5mm, F.Cu at (157.1, 86.5)
- added TP6: SCL_EEPROM, TestPoint:TestPoint_Pad_1.5x1.5mm, F.Cu at (160.2, 86.5)
- added TP7: 5V_Output, TestPoint:TestPoint_Pad_2.0x2.0mm, F.Cu at (139.2, 88.5)
- C1, C2: footprint Capacitor_SMD:C_0603_1608Metric -> Capacitor_SMD:C_0805_2012Metric
- C8: value 47uF -> 150uF; footprint Capacitor_SMD:CP_Elec_6.3x7.7 -> Capacitor_SMD:CP_Elec_10x12.5
- moved C8 28.4 mm to (146.0, 112.5), turned to -90 degrees
- moved R_Opt2 4.55 mm to (149.7, 131.5)
- moved R_Opt4 4.55 mm to (149.7, 123.5)
- moved R_Opt6 4.55 mm to (149.7, 127.5)
- moved R_Opt3 2.37 mm to (149.3, 104.0)
- moved R_Opt1 1.95 mm to (144.0, 86.2)
- moved R_Opt7 1.47 mm to (149.3, 101.0)
- moved C1 1.16 mm to (121.0, 106.5)
- moved C2 0.79 mm to (121.0, 104.5)
- moved EXT_POW1 0.58 mm to (135.9, 86.6)
- moved R4 0.58 mm to (135.9, 88.6)
- moved C3 0.24 mm to (121.3, 102.5)
- turned L1 to 90 degrees
Connections:
- J1 pad 10: /RXD -> unconnected-(J1-Pad10)
- J1 pad 3: /SDA -> unconnected-(J1-Pad3)
- J1 pad 5: /SCL -> unconnected-(J1-Pad5)
- J1 pad 8: /TXD -> unconnected-(J1-Pad8)
Routing:
- net GND: track 17.2 -> 160.8 mm
- net /ID_SCL_EEPROM: track 13.5 -> 25.3 mm
- net VCC: track 120.6 -> 113.2 mm
- net Net-(C4-Pad2): track 10.5 -> 17.2 mm
- net /Step1: track 55.8 -> 62.3 mm
- net /Dir2: track 32.4 -> 38.4 mm
- net /ID_SDA_EEPROM: track 9.13 -> 14.9 mm
- net /Dir1: track 66.6 -> 71.5 mm
- net +3V3: track 33.5 -> 28.9 mm
- net Net-(A1-Pad12): track 6.92 -> 11.1 mm
- net Net-(A1-Pad11): track 5.75 -> 9.37 mm
- net /Step2: track 41.0 -> 44.3 mm
- net Net-(A1-Pad10): track 5.15 -> 7.91 mm
- net Net-(A2-Pad12): track 13.5 -> 11.5 mm
- net Net-(R_Opt1-Pad2): track 6.54 -> 5.34 mm
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
Commit message: Make final changes
Parts:
- added G***: LOGO, iclr:iclr_logo, F.Cu at (116.5, 112.5)
- added G***: LOGO, iclr:Dom_License, B.Cu at (144.0, 105.0)
- TP2, TP4: moved to F.Cu
- moved TP4 17.2 mm to (158.2, 124.2), turned to 0 degrees
- moved TP2 16.6 mm to (158.2, 121.0), turned to 0 degrees
- moved BAT 7.15 mm to (123.5, 129.2), turned to 90 degrees
- moved C7 2.51 mm to (132.5, 121.2)
- moved TP5 0.75 mm to (157.1, 87.2)
- moved TP6 0.75 mm to (160.2, 87.2)
- moved C5 0.25 mm to (130.1, 87.2)
- renumbered J2 to BAT, J3 to DC, EXT_POW1 to EXT_POW, Fan1 to Fan, PI_POW1 to PI_POW, StepperConnector1 to Stepper1, StepperConnector2 to Stepper2
Connections:
- BAT pad 1: Net-(C6-Pad1) -> GND
- BAT pad 2: GND -> Net-(C6-Pad1)
Routing:
- net /Dir2: track 38.4 -> 54.1 mm, vias 0 -> 1
- net /Step2: track 44.3 -> 58.7 mm, vias 0 -> 1
- net GND: track 160.8 -> 162.8 mm
Other:
- board text added: "+ -"
- board text added: "0"
- board text added: "2Stepper2Driver"
- board text added: "4.7V-28V⎓"
- board text added: "JLCJLCJLCJLCJLCJLC"
- board text added: "Shitposted with <3 by Daniele Bella"
