File: Hardware/Dom-Turretto-Hat/Dom-Turretto-Hat.kicad_sch (KiCad schematic)
At the start: 10 parts, among them J1 Raspberry_Pi_2_3, U1 CAT24C32WI-GT3

Commit message: Made initial layout
Parts:
- H1, H2, H3, H4: footprint (none) -> MountingHole:MountingHole_2.7mm_M2.5
- JP1: footprint (none) -> Jumper:SolderJumper-2_P1.3mm_Open_RoundedPad1.0x1.5mm
- R1, R2, R3: footprint (none) -> Resistor_SMD:R_0603_1608Metric
- U1: footprint (none) -> iclr:SOIC127P600X175-8N
Changed lines of the file:
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@@
       (effects (font (size 1.27 1.27)) (justify right))
     )
-    (property "Footprint" "" (id 2) (at 57.15 34.29 0)
+    (property "Footprint" "MountingHole:MountingHole_2.7mm_M2.5" (id 2) (at 57.15 34.29 0)
       (effects (font (size 1.27 1.27)) hide)
     )
@@
     (property "Reference" "U1" (id 0) (at 64.77 85.09 0))
     (property "Value" "CAT24C32WI-GT3" (id 1) (at 64.77 87.63 0))
-    (property "Footprint" "" (id 2) (at 64.77 102.87 0)
+    (property "Footprint" "iclr:SOIC127P600X175-8N" (id 2) (at 64.77 102.87 0)
       (effects (font (size 1.27 1.27)) (justify left bottom) hide)
     )
@@
       (effects (font (size 1.27 1.27)) (justify left))
     )
-    (property "Footprint" "" (id 2) (at 69.85 153.67 0)
+    (property "Footprint" "Resistor_SMD:R_0603_1608Metric" (id 2) (at 69.85 153.67 0)
       (effects (font (size 1.27 1.27)) hide)
     )
@@
       (effects (font (size 1.27 1.27)) (justify left))
     )
-    (property "Footprint" "" (id 2) (at 57.15 39.37 0)
+    (property "Footprint" "MountingHole:MountingHole_2.7mm_M2.5" (id 2) (at 57.15 39.37 0)
       (effects (font (size 1.27 1.27)) hide)
     )
@@
       (effects (font (size 1.27 1.27)) (justify left))
     )
-    (property "Footprint" "" (id 2) (at 57.15 49.53 0)
+    (property "Footprint" "MountingHole:MountingHole_2.7mm_M2.5" (id 2) (at 57.15 49.53 0)
       (effects (font (size 1.27 1.27)) hide)
     )
@@
       (effects (font (size 1.27 1.27)) (justify right))
     )
-    (property "Footprint" "" (id 2) (at 57.15 44.45 0)
+    (property "Footprint" "MountingHole:MountingHole_2.7mm_M2.5" (id 2) (at 57.15 44.45 0)
       (effects (font (size 1.27 1.27)) hide)
     )
@@
       (effects (font (size 1.27 1.27)) (justify left))
     )
-    (property "Footprint" "" (id 2) (at 29.21 88.9 0)
+    (property "Footprint" "Jumper:SolderJumper-2_P1.3mm_Open_RoundedPad1.0x1.5mm" (id 2) (at 29.21 88.9 0)
       (effects (font (size 1.27 1.27)) hide)
     )
@@
       (effects (font (size 1.27 1.27)) (justify left))
     )
-    (property "Footprint" "" (id 2) (at 69.85 138.43 0)
+    (property "Footprint" "Resistor_SMD:R_0603_1608Metric" (id 2) (at 69.85 138.43 0)
       (effects (font (size 1.27 1.27)) hide)
     )
@@
       (effects (font (size 1.27 1.27)) (justify left))
     )
-    (property "Footprint" "" (id 2) (at 29.21 81.28 0)
+    (property "Footprint" "Resistor_SMD:R_0603_1608Metric" (id 2) (at 29.21 81.28 0)
       (effects (font (size 1.27 1.27)) hide)
     )
@@
       (reference "J2") (unit 1) (value "Conn_Coaxial") (footprint "Connector_Coaxial:SMA_Molex_73251-1153_EdgeMount_Horizontal")
     )
-    (path "/12e93b0c-a239-457f-b141-0c3b73a9b90a/f144d15c-aba2-4e4d-9f24-5cf24b835a90"
-      (reference "J3") (unit 1) (value "Barrel_Jack") (footprint "Connector_BarrelJack:BarrelJack_SwitchcraftConxall_RAPC10U_Horizontal")
+    (path "/12e93b0c-a239-457f-b141-0c3b73a9b90a/e7d03e9b-f8b8-44fa-a0bb-981b7bc05317"
+      (reference "J3") (unit 1) (value "Barrel_Jack_Switch") (footprint "Connector_BarrelJack:BarrelJack_Wuerth_6941xx301002")
     )
     (path "/12e93b0c-a239-457f-b141-0c3b73a9b90a/acb976e5-4afe-45ae-bace-6e56185fabf9"
