File: Hardware/Dom-Turretto-Hat/Dom-Turretto-Hat.kicad_sch (KiCad schematic)
At the start: 10 parts, among them J1 Raspberry_Pi_2_3, U1 CAT24C32WI-GT3

Commit message: Updated schematic
Other:
- removed sheet GPS
Changed lines of the file:
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@@
-    (stroke (width 0) (type default) (color 0 0 0 0))
-  )
-  (wire (pts (xy 224.79 63.5) (xy 227.33 63.5))
     (stroke (width 0) (type default) (color 0 0 0 0))
   )
@@
     (stroke (width 0) (type default) (color 0 0 0 0))
   )
-  (wire (pts (xy 224.79 60.96) (xy 227.33 60.96))
-    (stroke (width 0) (type default) (color 0 0 0 0))
-  )
   (wire (pts (xy 77.47 115.57) (xy 80.01 115.57))
     (stroke (width 0) (type default) (color 0 0 0 0))
@@
     (stroke (width 0) (type default) (color 0 0 0 0))
   )
-  (wire (pts (xy 224.79 68.58) (xy 227.33 68.58))
-    (stroke (width 0) (type default) (color 0 0 0 0))
-  )
   (wire (pts (xy 69.85 156.21) (xy 69.85 157.48))
     (stroke (width 0) (type default) (color 0 0 0 0))
@@
   )
   (wire (pts (xy 80.01 115.57) (xy 80.01 118.11))
-    (stroke (width 0) (type default) (color 0 0 0 0))
-  )
-  (wire (pts (xy 224.79 66.04) (xy 227.33 66.04))
     (stroke (width 0) (type default) (color 0 0 0 0))
   )
@@
     (effects (font (size 1.27 1.27)) (justify right bottom))
   )
-  (label "TXD" (at 224.79 66.04 180)
-    (effects (font (size 1.27 1.27)) (justify right bottom))
-  )
   (label "ID_SDA_EEPROM" (at 166.37 80.01 0)
     (effects (font (size 1.27 1.27)) (justify left bottom))
@@
     (effects (font (size 1.27 1.27)) (justify right bottom))
   )
-  (label "SDA" (at 224.79 60.96 180)
-    (effects (font (size 1.27 1.27)) (justify right bottom))
-  )
   (label "Dir1" (at 226.06 119.38 180)
     (effects (font (size 1.27 1.27)) (justify right bottom))
@@
     (effects (font (size 1.27 1.27)) (justify right bottom))
   )
-  (label "RXD" (at 224.79 68.58 180)
-    (effects (font (size 1.27 1.27)) (justify right bottom))
-  )
   (label "TXD" (at 120.65 80.01 180)
     (effects (font (size 1.27 1.27)) (justify right bottom))
@@
   )
   (label "Dir1" (at 120.65 113.03 180)
-    (effects (font (size 1.27 1.27)) (justify right bottom))
-  )
-  (label "SCL" (at 224.79 63.5 180)
     (effects (font (size 1.27 1.27)) (justify right bottom))
   )
@@
     )
   )
-  (sheet (at 227.33 58.42) (size 12.7 12.7) (fields_autoplaced)
-    (stroke (width 0.1524) (type solid) (color 0 0 0 0))
-    (fill (color 0 0 0 0.0000))
-    (property "Sheet name" "GPS" (id 0) (at 227.33 57.7084 0)
-      (effects (font (size 1.27 1.27)) (justify left bottom))
-    )
-    (property "Sheet file" "GPS.kicad_sch" (id 1) (at 227.33 71.7046 0)
-      (effects (font (size 1.27 1.27)) (justify left top))
-    )
-    (pin "RXD" input (at 227.33 68.58 180)
-      (effects (font (size 1.27 1.27)) (justify left))
-    )
-    (pin "SDA" input (at 227.33 60.96 180)
-      (effects (font (size 1.27 1.27)) (justify left))
-    )
-    (pin "SCL" input (at 227.33 63.5 180)
-      (effects (font (size 1.27 1.27)) (justify left))
-    )
-    (pin "TXD" input (at 227.33 66.04 180)
-      (effects (font (size 1.27 1.27)) (justify left))
-    )
-  )
   (sheet_instances
     (path "/" (page "1"))
-    (path "/c8c14f7c-55ef-44f2-9b65-a499409017e1" (page "2"))
     (path "/12e93b0c-a239-457f-b141-0c3b73a9b90a" (page "3"))
     (path "/28fd1fbc-026b-4dd2-b303-4aef81adb474" (page "4"))
@@
       (reference "#PWR08") (unit 1) (value "GND") (footprint "")
     )
-    (path "/c8c14f7c-55ef-44f2-9b65-a499409017e1/e4566a45-8e06-47ea-a935-fa62dd278c90"
-      (reference "#PWR09") (unit 1) (value "+3V3") (footprint "")
-    )
-    (path "/c8c14f7c-55ef-44f2-9b65-a499409017e1/899f9b0d-851b-40b2-95d9-0bf4320cfc7f"
-      (reference "#PWR010") (unit 1) (value "+3V3") (footprint "")
-    )
-    (path "/c8c14f7c-55ef-44f2-9b65-a499409017e1/451985fb-27af-4988-a96b-5b9018357ef6"
-      (reference "#PWR011") (unit 1) (value "GND") (footprint "")
-    )
-    (path "/c8c14f7c-55ef-44f2-9b65-a499409017e1/d58204f5-4242-4763-8399-6e93946856c1"
-      (reference "#PWR012") (unit 1) (value "GND") (footprint "")
-    )
     (path "/12e93b0c-a239-457f-b141-0c3b73a9b90a/462f3a13-0050-4845-84df-8be913b4f9b0"
       (reference "#PWR013") (unit 1) (value "VCC") (footprint "")
@@
       (reference "A2") (unit 1) (value "Pololu_Breakout_A4988") (footprint "Module:Pololu_Breakout-16_15.2x20.3mm")
     )
-    (path "/c8c14f7c-55ef-44f2-9b65-a499409017e1/4fb87244-379d-4e75-94c2-9521bcc0ec81"
-      (reference "C1") (unit 1) (value "10nF") (footprint "Capacitor_SMD:C_0603_1608Metric")
-    )
     (path "/12e93b0c-a239-457f-b141-0c3b73a9b90a/ec276c8a-eb48-440f-b539-492777d28831"
       (reference "C2") (unit 1) (value "22uF") (footprint "Capacitor_SMD:C_0603_1608Metric")
@@
       (reference "J1") (unit 1) (value "Raspberry_Pi_2_3") (footprint "Connector_PinSocket_2.54mm:PinSocket_2x20_P2.54mm_Vertical")
     )
-    (path "/c8c14f7c-55ef-44f2-9b65-a499409017e1/6a180251-fad0-4435-9a6c-41f5e820bcf1"
-      (reference "J2") (unit 1) (value "Conn_Coaxial") (footprint "Connector_Coaxial:SMA_Molex_73251-1153_EdgeMount_Horizontal")
-    )
     (path "/12e93b0c-a239-457f-b141-0c3b73a9b90a/e7d03e9b-f8b8-44fa-a0bb-981b7bc05317"
       (reference "J3") (unit 1) (value "Barrel_Jack_Switch") (footprint "Connector_BarrelJack:BarrelJack_Wuerth_6941xx301002")
@@
       (reference "JP1") (unit 1) (value "SolderJumper_2_Open") (footprint "Jumper:SolderJumper-2_P1.3mm_Open_RoundedPad1.0x1.5mm")
     )
-    (path "/c8c14f7c-55ef-44f2-9b65-a499409017e1/d6c763e2-1952-4281-9868-501fafa3b154"
-      (reference "L1") (unit 1) (value "27nH") (footprint "Inductor_SMD:L_0603_1608Metric")
-    )
     (path "/12e93b0c-a239-457f-b141-0c3b73a9b90a/89b193d6-28e4-4647-a3aa-6b8779163e05"
       (reference "L2") (unit 1) (value "29uH") (footprint "Inductor_SMD:L_12x12mm_H8mm")
@@
       (reference "R3") (unit 1) (value "3.9k") (footprint "Resistor_SMD:R_0603_1608Metric")
     )
-    (path "/c8c14f7c-55ef-44f2-9b65-a499409017e1/d53051b6-ebe9-4558-9887-00e35561baeb"
-      (reference "R4") (unit 1) (value "10K") (footprint "Resistor_SMD:R_0603_1608Metric")
-    )
-    (path "/c8c14f7c-55ef-44f2-9b65-a499409017e1/8a505506-ea00-4e73-916e-6375c9e26bd9"
-      (reference "R5") (unit 1) (value "10") (footprint "Resistor_SMD:R_0603_1608Metric")
-    )
     (path "/12e93b0c-a239-457f-b141-0c3b73a9b90a/fdd22b43-7b45-4042-a6f9-6eedcac49126"
       (reference "R6") (unit 1) (value "1k") (footprint "Resistor_SMD:R_0603_1608Metric")
@@
       (reference "R_Opt6") (unit 1) (value "10k") (footprint "Resistor_SMD:R_0603_1608Metric")
     )
-    (path "/28fd1fbc-026b-4dd2-b303-4aef81adb474/7b127ce6-8a99-4db8-b9ae-9816ab607482"
-      (reference "Stepper1") (unit 1) (value "Conn_01x04_Male") (footprint "Connector_PinHeader_2.54mm:PinHeader_1x04_P2.54mm_Vertical")
-    )
-    (path "/28fd1fbc-026b-4dd2-b303-4aef81adb474/4d5b4119-b68b-4420-a981-41d30b5b527a"
-      (reference "Stepper2") (unit 1) (value "Conn_01x04_Male") (footprint "Connector_PinHeader_2.54mm:PinHeader_1x04_P2.54mm_Vertical")
+    (path "/28fd1fbc-026b-4dd2-b303-4aef81adb474/42207e46-1957-49ff-9e9f-2c15c2c27eb3"
+      (reference "StepperConnector1") (unit 1) (value "Screw_Terminal_01x04") (footprint "TerminalBlock_TE-Connectivity:TerminalBlock_TE_282834-4_1x04_P2.54mm_Horizontal")
+    )
+    (path "/28fd1fbc-026b-4dd2-b303-4aef81adb474/d265b409-1fc4-41c9-b7f5-c0ea5c831019"
+      (reference "StepperConnector2") (unit 1) (value "Screw_Terminal_01x04") (footprint "TerminalBlock_TE-Connectivity:TerminalBlock_TE_282834-4_1x04_P2.54mm_Horizontal")
     )
     (path "/2502caee-d955-453d-8eae-fa5e480fab5f"
       (reference "U1") (unit 1) (value "CAT24C32WI-GT3") (footprint "iclr:SOIC127P600X175-8N")
     )
-    (path "/c8c14f7c-55ef-44f2-9b65-a499409017e1/5c054c83-012c-4e45-901b-5550fc59a449"
-      (reference "U2") (unit 1) (value "MAX-M8Q") (footprint "RF_GPS:ublox_MAX")
-    )
     (path "/12e93b0c-a239-457f-b141-0c3b73a9b90a/07f473c2-dbb9-400c-8bca-062c33fea70b"

Commit message: Update components
Parts:
- added H5, H6: MountingHole, MountingHole:MountingHole_2.7mm_M2.5, symbol Mechanical:MountingHole
Connections:
- no-connect marks 2 -> 4
Changed lines of the file:
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@@
   (no_connect (at 146.05 69.85))
   (no_connect (at 148.59 69.85))
+  (no_connect (at -303.53 -21.59))
+  (no_connect (at 232.41 88.9))
   (wire (pts (xy 52.07 105.41) (xy 52.07 107.95))
     (stroke (width 0) (type default) (color 0 0 0 0))
@@
     )
     (property "Datasheet" "~" (id 3) (at 57.15 39.37 0)
+      (effects (font (size 1.27 1.27)) hide)
+    )
+  )
+  (symbol (lib_id "Mechanical:MountingHole") (at 57.15 54.61 90) (unit 1)
+    (in_bom yes) (on_board yes) (fields_autoplaced)
+    (property "Reference" "H5" (id 0) (at 59.69 53.3399 90)
+      (effects (font (size 1.27 1.27)) (justify right))
+    )
+    (property "Value" "MountingHole" (id 1) (at 59.69 55.8799 90)
+      (effects (font (size 1.27 1.27)) (justify right))
+    )
+    (property "Footprint" "MountingHole:MountingHole_2.7mm_M2.5" (id 2) (at 57.15 54.61 0)
+      (effects (font (size 1.27 1.27)) hide)
+    )
+    (property "Datasheet" "~" (id 3) (at 57.15 54.61 0)
+      (effects (font (size 1.27 1.27)) hide)
+    )
+  )
+  (symbol (lib_id "Mechanical:MountingHole") (at 57.15 59.69 0) (unit 1)
+    (in_bom yes) (on_board yes) (fields_autoplaced)
+    (property "Reference" "H6" (id 0) (at 59.69 58.4199 0)
+      (effects (font (size 1.27 1.27)) (justify left))
+    )
+    (property "Value" "MountingHole" (id 1) (at 59.69 60.9599 0)
+      (effects (font (size 1.27 1.27)) (justify left))
+    )
+    (property "Footprint" "MountingHole:MountingHole_2.7mm_M2.5" (id 2) (at 57.15 59.69 0)
+      (effects (font (size 1.27 1.27)) hide)
+    )
+    (property "Datasheet" "~" (id 3) (at 57.15 59.69 0)
       (effects (font (size 1.27 1.27)) hide)
     )
@@
       (reference "#PWR018") (unit 1) (value "GND") (footprint "")
     )
-    (path "/12e93b0c-a239-457f-b141-0c3b73a9b90a/77d8b42a-8f24-44ab-896a-843f58a19ca6"
-      (reference "#PWR019") (unit 1) (value "VCC") (footprint "")
-    )
-    (path "/12e93b0c-a239-457f-b141-0c3b73a9b90a/279b3b38-0ca0-4170-b0e5-b4a71141ec1d"
-      (reference "#PWR020") (unit 1) (value "VCC") (footprint "")
-    )
     (path "/12e93b0c-a239-457f-b141-0c3b73a9b90a/ef21a8b1-2228-4fe0-8e53-070fce64f3d9"
       (reference "#PWR021") (unit 1) (value "GND") (footprint "")
     )
-    (path "/12e93b0c-a239-457f-b141-0c3b73a9b90a/5d29948f-b092-436d-8569-e312278ab4b8"
-      (reference "#PWR022") (unit 1) (value "~") (footprint "")
-    )
-    (path "/12e93b0c-a239-457f-b141-0c3b73a9b90a/0a30e9f2-6e1b-4ec8-8dfb-97bb7330560b"
-      (reference "#PWR023") (unit 1) (value "GND") (footprint "")
-    )
-    (path "/12e93b0c-a239-457f-b141-0c3b73a9b90a/0d3f8564-cd5b-4df8-9d76-9b7db354d95d"
-      (reference "#PWR024") (unit 1) (value "VCC") (footprint "")
-    )
-    (path "/12e93b0c-a239-457f-b141-0c3b73a9b90a/5cb16795-6314-4e78-a6d5-607bc482b6b8"
-      (reference "#PWR025") (unit 1) (value "VCC") (footprint "")
-    )
     (path "/12e93b0c-a239-457f-b141-0c3b73a9b90a/edde2f9a-acc0-48b1-bb93-b02152a9c39d"
       (reference "#PWR026") (unit 1) (value "VCC") (footprint "")
@@
       (reference "#PWR038") (unit 1) (value "+5V") (footprint "")
     )
-    (path "/28fd1fbc-026b-4dd2-b303-4aef81adb474/55303a26-0455-4f2e-a196-ba787a54142b"
-      (reference "#PWR039") (unit 1) (value "+3V3") (footprint "")
-    )
-    (path "/28fd1fbc-026b-4dd2-b303-4aef81adb474/a9f6ebbd-02a8-4b2b-a4c5-15a1790ac4de"
-      (reference "#PWR040") (unit 1) (value "+3V3") (footprint "")
-    )
-    (path "/28fd1fbc-026b-4dd2-b303-4aef81adb474/fc935fe0-8219-452b-9c6c-b59c1b60386d"
-      (reference "#PWR041") (unit 1) (value "+3V3") (footprint "")
-    )
-    (path "/28fd1fbc-026b-4dd2-b303-4aef81adb474/c1ff0eb3-9302-47ed-b15d-9e16331b840e"
-      (reference "#PWR042") (unit 1) (value "+3V3") (footprint "")
-    )
     (path "/28fd1fbc-026b-4dd2-b303-4aef81adb474/b4594279-7934-4f54-9da4-b5ed23f051f5"
       (reference "#PWR043") (unit 1) (value "GND") (footprint "")
@@
       (reference "#PWR044") (unit 1) (value "GND") (footprint "")
     )
-    (path "/28fd1fbc-026b-4dd2-b303-4aef81adb474/0093ac4f-b653-4c0f-be83-e1871bb4f9fa"
-      (reference "#PWR045") (unit 1) (value "+3V3") (footprint "")
-    )
-    (path "/28fd1fbc-026b-4dd2-b303-4aef81adb474/dbad90c2-b64e-4729-99dc-c80264470e92"
-      (reference "#PWR046") (unit 1) (value "+3V3") (footprint "")
-    )
-    (path "/28fd1fbc-026b-4dd2-b303-4aef81adb474/020c7563-050d-4993-a33e-5454a0d9355c"
-      (reference "#PWR047") (unit 1) (value "+3V3") (footprint "")
-    )
-    (path "/28fd1fbc-026b-4dd2-b303-4aef81adb474/46550aaa-c0b4-4d92-bd6b-7e22e8b199b7"
-      (reference "#PWR048") (unit 1) (value "+3V3") (footprint "")
-    )
     (path "/28fd1fbc-026b-4dd2-b303-4aef81adb474/d86fb79d-c0ac-434f-ba25-b2b1233a8f26"
       (reference "#PWR049") (unit 1) (value "GND") (footprint "")
@@
       (reference "#PWR054") (unit 1) (value "GND") (footprint "")
     )
+    (path "/12e93b0c-a239-457f-b141-0c3b73a9b90a/16d2fdc2-babd-49b7-b3f4-8ebee5bb6b22"
+      (reference "#PWR0101") (unit 1) (value "VCC") (footprint "")
+    )
+    (path "/12e93b0c-a239-457f-b141-0c3b73a9b90a/76776ac9-01ea-4972-9d87-dd0a762af3c9"
+      (reference "#PWR0102") (unit 1) (value "GND") (footprint "")
+    )
+    (path "/28fd1fbc-026b-4dd2-b303-4aef81adb474/a67e1f19-66f8-4d89-a414-1dd966045ad0"
+      (reference "#PWR0103") (unit 1) (value "+5V") (footprint "")
+    )
+    (path "/28fd1fbc-026b-4dd2-b303-4aef81adb474/9dc995cd-8c94-45d3-a4e1-d727a2822c72"
+      (reference "#PWR0104") (unit 1) (value "+5V") (footprint "")
+    )
+    (path "/28fd1fbc-026b-4dd2-b303-4aef81adb474/26251c45-5edc-47f5-bbe9-a3fa40eb07cf"
+      (reference "#PWR0105") (unit 1) (value "+5V") (footprint "")
+    )
+    (path "/28fd1fbc-026b-4dd2-b303-4aef81adb474/b601569f-09f4-4cef-b542-0b3745596966"
+      (reference "#PWR0106") (unit 1) (value "+5V") (footprint "")
+    )
+    (path "/28fd1fbc-026b-4dd2-b303-4aef81adb474/a83d4d91-ae71-431a-9357-40ec7588a902"
+      (reference "#PWR0107") (unit 1) (value "+5V") (footprint "")
+    )
+    (path "/28fd1fbc-026b-4dd2-b303-4aef81adb474/6788054c-34eb-4edd-af0a-8aff4765f859"
+      (reference "#PWR0108") (unit 1) (value "+5V") (footprint "")
+    )
+    (path "/28fd1fbc-026b-4dd2-b303-4aef81adb474/e9bf3fe6-e1cc-4b8d-bbb8-700e183aad7b"
+      (reference "#PWR0109") (unit 1) (value "+5V") (footprint "")
+    )
+    (path "/28fd1fbc-026b-4dd2-b303-4aef81adb474/35f07658-fb63-46ec-8bc3-dc98eda80c44"
+      (reference "#PWR0110") (unit 1) (value "+5V") (footprint "")
+    )
     (path "/28fd1fbc-026b-4dd2-b303-4aef81adb474/84977e32-dddb-4234-a567-e1e9c75d8f8b"
       (reference "A1") (unit 1) (value "Pololu_Breakout_A4988") (footprint "Module:Pololu_Breakout-16_15.2x20.3mm")
@@
       (reference "H4") (unit 1) (value "MountingHole") (footprint "MountingHole:MountingHole_2.7mm_M2.5")
     )
+    (path "/33c57a88-3c0b-42cc-b00b-b98c1db847d9"
+      (reference "H5") (unit 1) (value "MountingHole") (footprint "MountingHole:MountingHole_2.7mm_M2.5")
+    )
+    (path "/4ad87c7f-b1c1-433e-a5bb-e4fec5b6bea0"
+      (reference "H6") (unit 1) (value "MountingHole") (footprint "MountingHole:MountingHole_2.7mm_M2.5")
+    )
     (path "/61fae217-e18a-4e68-8630-42cc06a8ba2f"
       (reference "J1") (unit 1) (value "Raspberry_Pi_2_3") (footprint "Connector_PinSocket_2.54mm:PinSocket_2x20_P2.54mm_Vertical")
@@
     )
     (path "/12e93b0c-a239-457f-b141-0c3b73a9b90a/acb976e5-4afe-45ae-bace-6e56185fabf9"
-      (reference "J4") (unit 1) (value "Conn_01x02") (footprint "Connector_AMASS:AMASS_XT60-M_1x02_P7.20mm_Vertical")
+      (reference "J4") (unit 1) (value "Conn_01x02") (footprint "Connector_AMASS:AMASS_XT60-F_1x02_P7.20mm_Vertical")
     )
     (path "/a4265e2c-06a9-41da-b42d-91d87bbe6b18"
@@
       (reference "PI_POW1") (unit 1) (value "LED") (footprint "LED_SMD:LED_0603_1608Metric")
     )
+    (path "/12e93b0c-a239-457f-b141-0c3b73a9b90a/87939eb2-1100-49c2-9486-7d16102560a9"
+      (reference "Q1") (unit 1) (value "RSJ250P10TL") (footprint "Package_TO_SOT_SMD:TO-263-3_TabPin2")
+    )
+    (path "/12e93b0c-a239-457f-b141-0c3b73a9b90a/d771511f-d16d-4f8b-8935-04481cf37b67"
+      (reference "Q2") (unit 1) (value "RSJ250P10TL") (footprint "Package_TO_SOT_SMD:TO-263-3_TabPin2")
+    )
     (path "/e3cbd370-7c22-4222-878e-9ad9b35baaf2"
       (reference "R1") (unit 1) (value "10k") (footprint "Resistor_SMD:R_0603_1608Metric")
@@
       (reference "R3") (unit 1) (value "3.9k") (footprint "Resistor_SMD:R_0603_1608Metric")
     )
+    (path "/12e93b0c-a239-457f-b141-0c3b73a9b90a/9880ee0b-bf61-4137-87f3-1f80c379eeea"
+      (reference "R4") (unit 1) (value "470k") (footprint "Resistor_SMD:R_0603_1608Metric")
+    )
     (path "/12e93b0c-a239-457f-b141-0c3b73a9b90a/fdd22b43-7b45-4042-a6f9-6eedcac49126"
       (reference "R6") (unit 1) (value "1k") (footprint "Resistor_SMD:R_0603_1608Metric")
@@
       (reference "U1") (unit 1) (value "CAT24C32WI-GT3") (footprint "iclr:SOIC127P600X175-8N")
     )
+    (path "/12e93b0c-a239-457f-b141-0c3b73a9b90a/3088a965-e082-4091-b39a-e0cabeff142b"
+      (reference "U2") (unit 1) (value "LTC4412xS6") (footprint "Package_TO_SOT_SMD:TSOT-23-6")
+    )
     (path "/12e93b0c-a239-457f-b141-0c3b73a9b90a/07f473c2-dbb9-400c-8bca-062c33fea70b"
       (reference "U3") (unit 1) (value "LM22679TJ-5.0{slash}NOPB") (footprint "iclr:TO127P1401X200-7N")
     )
-    (path "/12e93b0c-a239-457f-b141-0c3b73a9b90a/61250057-4a71-4881-93cc-88ea1d9c9a67"
-      (reference "U4") (unit 1) (value "LTC4451AV#TRMPBF") (footprint "iclr:IC_LTC4451AV#TRMPBF")
-    )
-    (path "/12e93b0c-a239-457f-b141-0c3b73a9b90a/d385e05a-2105-4728-bc50-3a756fa000d3"
-      (reference "U5") (unit 1) (value "LTC4451AV#TRMPBF") (footprint "iclr:IC_LTC4451AV#TRMPBF")
-    )
     (path "/12e93b0c-a239-457f-b141-0c3b73a9b90a/eb5b72c6-f2a4-4154-bfb1-f9f38e61bca2"
